Commit message: Merged fix to stop call to grasp execution service if no grasp plan planned/no objects, and overhaul GraspScene to be templated instead for easy implementation

File: scenes/ur5_2f_test/urdf/scene.urdf.xacro (robot description, xacro)
@@ -24,5 +24,5 @@
  <xacro:arg name="use_nominal_extrinsics" default="true" />
  <xacro:sensor_d415 parent="table_" use_nominal_extrinsics="$(arg use_nominal_extrinsics)">
-    <origin xyz="-0.58 0.225 0.65" rpy="3.14159 1.57079506 0"/>
+    <origin xyz="-0.58 0.12 0.655" rpy="0 1.57079506 0"/>
  </xacro:sensor_d415>
  <link name="camera_frame" />
